File: kicad.d/pnp_flwng_npn/kicad_23_dec_2021-a/kicad_23_dec_2021-a.sch (KiCad schematic (older format))
At the start: 0 parts

Commit message: new project files
	modified:   kicad_23_dec_2021-a-cache.lib
	modified:   kicad_23_dec_2021-a.pro
	modified:   kicad_23_dec_2021-a.sch
	new file:   kicad_23_dec_2021-a.svg
	new file:   kicad_23_dec_2021-a_0113z.svg
	new file:   kicad_23_dec_2021-b-cache.lib
	new file:   kicad_23_dec_2021-b.sch

On branch dvlp-aa
Parts:
- added D1, D? (x2): LED, symbol Device:LED
- added MES1: 1.544 mA, symbol Device:Amperemeter_AC
- added MES2: 92.905 uA, symbol Device:Amperemeter_AC
- added MES?: unknown, symbol Device:Amperemeter_AC
- added MES?: 3.582 mA, symbol Device:Amperemeter_AC
- added MES?: 1.534 mA, symbol Device:Amperemeter_AC
- added MES?: 4.326 mA, symbol Device:Amperemeter_AC
- added MES?: 651 uA, symbol Device:Amperemeter_AC
- added MES?: 5.116 mA, symbol Device:Amperemeter_AC
- added MES?: 4.233 mA, symbol Device:Amperemeter_AC
- added Q1, Q?: 2N3904, Package_TO_SOT_THT:TO-92_Inline, symbol Transistor_BJT:2N3904
- added Q2, Q?: 2N3906, Package_TO_SOT_THT:TO-92_Inline, symbol Transistor_BJT:2N3906
- added R1, R? (x2): 47k, symbol Device:R_US
- added R2, R3, R? (x2): 1k, symbol Device:R_US
- added R4, R? (x2): 2.2k, symbol Device:R_US
- added U?: ULN2803A, symbol Transistor_Array:ULN2803A
- added V1, V? (x2): VPULSE, symbol Simulation_SPICE:VPULSE
Connections:
- net labels added: +3.3V, GNDREF
- wire segments 0 -> 28
Other:
- note removed: "lmnop"
