File: kicad.d/pnp_flwng_npn/kicad_24_dec_2021-c/kicad_24_dec_2021-c.sch (KiCad schematic (older format))
At the start: 20 parts

Commit message: many details added
Parts:
- added D?: D_Schottky, symbol Device:D_Schottky
- added MES?: 675.371 mV, symbol Device:Voltmeter_DC
- added MES?: VCE 418.47 mV, symbol Device:Voltmeter_DC
- added MES_B-?: 14.179 mA, symbol Device:Amperemeter_AC
- added MES_B-?: 139.31 uA (just saturated), symbol Device:Amperemeter_AC
- added MES_B-? (x2): 637.692 uA, symbol Device:Amperemeter_AC
- added Q?: 2N3906, Package_TO_SOT_THT:TO-92_Inline, symbol Transistor_BJT:2N3906
- added R?: 668/332 1k, symbol Device:R_Variable_US
- added R_B-?: 1k, symbol Device:R_US
- added R_B-?: 6.8k, symbol Device:R_US
- added SW_B-?: SW_SPDT, symbol Switch:SW_SPDT
- added U?: ULN2803A, symbol Transistor_Array:ULN2803A
- MES?: value 122.381 mV -> VCE 418.47 mV
- MES?: value 1.852 V -> 1.817 V
- MES_B-33: value 386.217 uA -> 248.373 uA
- MES_B-77: value 20.168 mA -> 13.931 mA
Connections:
- wire segments 34 -> 63
Other:
- note added: "SPDT == GPIO pin"
- moved on the sheet: D1, D?, MES?, MES_B-144, MES_B-33, MES_B-55, MES_B-77, MES_B-88, MES_B-?, Pulsed_A, Q_B-33, Q_B-?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

Commit message: for commit 6e3ff39
Parts:
- D?: value D_Schottky -> Schottky
Other:
- note added: "171.435 nA"
Changed lines of the file:
@@
 P 2000 2000
 F 0 "D?" V 2046 1920 50  0000 R CNN
-F 1 "D_Schottky" V 1955 1920 50  0000 R CNN
+F 1 "Schottky" V 1950 2450 50  0001 R CNN
 F 2 "" H 2000 2000 50  0001 C CNN
 F 3 "~" H 2000 2000 50  0001 C CNN
@@
 	-1   0    0    -1
 $EndComp
+Text Notes 3450 2050 0    50   ~ 0
+171.435 nA
 $EndSCHEMATC

Commit message: Refinements and Reference clean-ups.
	modified:   kicad_24_dec_2021-c.png
	modified:   kicad_24_dec_2021-c.sch
	modified:   kicad_24_dec_2021-c.svg

On branch dvlp-aa
Parts:
- removed MES?: VCE 418.47 mV, symbol Device:Voltmeter_DC
- removed MES_B-55: 20.554 mA, symbol Device:Amperemeter_AC
- removed Q_B-33: 2N3904, Package_TO_SOT_THT:TO-92_Inline, symbol Transistor_BJT:2N3904
- MES_7: renamed from MES_B-88; value 386.217 uA -> 248.373 uA
- MES_8: renamed from MES_B-144; value -5.09 pA -> 4.854 pA
- gave numbers to parts that had none: 21
- renumbered D1 to D2, MES_B-77 to MES_6, MES_B-33 to MES_9, R_B-2 to R4, R_B-1 to R5
Connections:
- wire segments 63 -> 55
Changed lines of the file:
@@
 $EndDescr
 $Comp
-L Device:Amperemeter_AC MES_B-77
+L Device:Amperemeter_AC MES_6
 U 1 1 61D27D60
 P 5500 4000
-F 0 "MES_B-77" H 5700 4050 50  0000 L CNN
+F 0 "MES_6" H 5700 4050 50  0000 L CNN
 F 1 "13.931 mA" H 5700 3900 50  0000 L CNN
 F 2 "" V 5500 4100 50  0001 C CNN
@@
 $EndComp
 $Comp
-L Device:Amperemeter_AC MES_B-55
-U 1 1 61CF8DDE
-P 8150 1700
-F 0 "MES_B-55" H 8550 1750 50  0000 C CNN
-F 1 "20.554 mA" H 8750 1600 50  0000 R CNN
-F 2 "" V 8150 1800 50  0001 C CNN
-F 3 "~" V 8150 1800 50  0001 C CNN
-	1    8150 1700
-	1    0    0    -1
-$EndComp
-$Comp
-L Transistor_BJT:2N3904 Q_B-33
-U 1 1 61C80D14
-P 9150 2100
-F 0 "Q_B-33" H 9400 2150 50  0000 L CNN
-F 1 "2N3904" H 9400 2000 50  0000 L CNN
-F 2 "Package_TO_SOT_THT:TO-92_Inline" H 9350 2025 50  0001 L CIN
-F 3 "https://www.onsemi.com/pub/Collateral/2N3903-D.PDF" H 9150 2100 50  0001 L CNN
-	1    9150 2100
-	1    0    0    -1
-$EndComp
-$Comp
-L Device:LED D1
+L Device:LED D2
 U 1 1 61C80D07
 P 5500 3500
-F 0 "D1" V 5539 3382 50  0000 R CNN
+F 0 "D2" V 5539 3382 50  0000 R CNN
 F 1 "LED" V 5448 3382 50  0000 R CNN
 F 2 "" H 5500 3500 50  0001 C CNN
@@
 $EndComp
 $Comp
-L power:GNDREF #PWR?
-U 1 1 61C80CF5
-P 8150 1900
-F 0 "#PWR?" H 8150 1650 50  0001 C CNN
-F 1 "GNDREF" H 8155 1727 50  0001 C CNN
-F 2 "" H 8150 1900 50  0001 C CNN
-F 3 "" H 8150 1900 50  0001 C CNN
-	1    8150 1900
-	1    0    0    -1
-$EndComp
-$Comp
-L Device:R_US R_B-1
+L Device:R_US R5
 U 1 1 61C80CDD
 P 3200 5050
-F 0 "R_B-1" V 3405 5050 50  0000 C CNN
+F 0 "R5" V 3405 5050 50  0000 C CNN
 F 1 "6.8k" V 3314 5050 50  0000 C CNN
 F 2 "" V 3240 5040 50  0001 C CNN
@@
 $EndComp
 $Comp
-L Device:Amperemeter_AC MES_B-144
+L Device:Amperemeter_AC MES_8
 U 1 1 61D1013E
 P 2100 5400
-F 0 "MES_B-144" H 1700 5250 50  0000 C CNN
-F 1 "-5.09 pA" H 2650 5450 50  0000 R CNN
+F 0 "MES_8" H 1700 5250 50  0000 C CNN
+F 1 "4.854 pA" H 2650 5450 50  0000 R CNN
 F 2 "" V 2100 5500 50  0001 C CNN
 F 3 "~" V 2100 5500 50  0001 C CNN
@@
 $EndComp
 $Comp
-L Device:Amperemeter_AC MES_B-88
+L Device:Amperemeter_AC MES_7
 U 1 1 61D16E82
 P 2100 4700
-F 0 "MES_B-88" H 2450 4550 50  0000 C CNN
-F 1 "386.217 uA" H 1950 4800 50  0000 R CNN
+F 0 "MES_7" H 2450 4550 50  0000 C CNN
+F 1 "248.373 uA" H 1950 4800 50  0000 R CNN
 F 2 "" V 2100 4800 50  0001 C CNN
 F 3 "~" V 2100 4800 50  0001 C CNN
@@
 	2100 5150 2100 5200
 $Comp
-L Device:Amperemeter_AC MES_B-33
+L Device:Amperemeter_AC MES_9
 U 1 1 61C9332E
 P 3750 5050
-F 0 "MES_B-33" V 3950 5050 50  0000 C CNN
+F 0 "MES_9" V 3950 5050 50  0000 C CNN
 F 1 "248.373 uA" V 3550 5050 50  0000 C CNN
 F 2 "" V 3750 5150 50  0001 C CNN
@@
 	3950 5050 4200 5050
 $Comp
-L Device:LED D?
+L Device:LED D_B-1
 U 1 1 61E20E38
 P 10200 2000
-F 0 "D?" V 10239 1882 50  0000 R CNN
+F 0 "D_B-1" V 10239 1882 50  0000 R CNN
 F 1 "LED" V 10148 1882 50  0000 R CNN
 F 2 "" H 10200 2000 50  0001 C CNN
@@
 $EndComp
 $Comp
-L Device:R_US R_B-?
+L Device:R_US R_B-1
 U 1 1 61E20E3E
 P 10200 1600
-F 0 "R_B-?" H 10300 1700 50  0000 L CNN
+F 0 "R_B-1" H 10300 1700 50  0000 L CNN
 F 1 "150" H 10300 1500 50  0000 L CNN
 F 2 "" V 10240 1590 50  0001 C CNN
@@
 	10200 1750 10200 1850
 $Comp
-L Device:Amperemeter_AC MES_B-?
+L Device:Amperemeter_AC MES_B-1
 U 1 1 61E2793C
 P 10200 2450
-F 0 "MES_B-?" H 10600 2500 50  0000 C CNN
+F 0 "MES_B-1" H 10600 2500 50  0000 C CNN
 F 1 "20.959 mA" H 10800 2350 50  0000 R CNN
 F 2 "" V 10200 2550 50  0001 C CNN
@@
 $EndComp
 $Comp
-L Device:Voltmeter_DC MES?
-U 1 1 61E31E3B
-P 8900 1150
-F 0 "MES?" H 9053 1196 50  0000 L CNN
-F 1 "VCE 418.47 mV" H 9053 1105 50  0000 L CNN
-F 2 "" V 8900 1250 50  0001 C CNN
-F 3 "~" V 8900 1250 50  0001 C CNN
-	1    8900 1150
-	1    0    0    -1
-$EndComp
-$Comp
-L Device:Voltmeter_DC MES?
+L Device:Voltmeter_DC MES_5
 U 1 1 61E345A0
 P 6250 3500
-F 0 "MES?" H 6403 3546 50  0000 L CNN
+F 0 "MES_5" H 6403 3546 50  0000 L CNN
 F 1 "1.817 V" H 6403 3455 50  0000 L CNN
 F 2 "" V 6250 3600 50  0001 C CNN
@@
 $EndComp
 Wire Wire Line
-	8900 950  8900 850
-Wire Wire Line
-	8900 850  8150 850
-Wire Wire Line
-	8900 1350 8900 1450
-Wire Wire Line
-	8900 1450 8150 1450
-Wire Wire Line
-	8150 1450 8150 1350
-Wire Wire Line
 	5500 3250 6250 3250
 Wire Wire Line
@@
 Wire Wire Line
 	5500 3750 5500 3800
-Wire Wire Line
-	8150 800  8150 850
-Connection ~ 8150 850
-Wire Wire Line
-	8150 850  8150 950
-Wire Wire Line
-	8150 1500 8150 1450
-Connection ~ 8150 1450
 Text Notes 7950 6900 0    50   ~ 10
 Darlington NPN to be included\n24 Dec 2021  11:00:24z
 $Comp
-L Transistor_BJT:2N3904 Q_B-?
+L Transistor_BJT:2N3904 Q_C-1
 U 1 1 61E9ABBA
 P 10100 5650
-F 0 "Q_B-?" H 10350 5700 50  0000 L CNN
+F 0 "Q_C-1" H 10350 5700 50  0000 L CNN
 F 1 "2N3904" H 10350 5550 50  0000 L CNN
 F 2 "Package_TO_SOT_THT:TO-92_Inline" H 10300 5575 50  0001 L CIN
@@
 $EndComp
 $Comp
-L Device:LED D?
+L Device:LED D_C-1
 U 1 1 61E9ABC0
 P 10200 5150
-F 0 "D?" V 10239 5032 50  0000 R CNN
+F 0 "D_C-1" V 10239 5032 50  0000 R CNN
 F 1 "LED" V 10148 5032 50  0000 R CNN
 F 2 "" H 10200 5150 50  0001 C CNN
@@
 $EndComp
 $Comp
-L Device:R_US R_B-?
+L Device:R_US R_C-2
 U 1 1 61E9ABCC
 P 10200 4700
-F 0 "R_B-?" H 10300 4800 50  0000 L CNN
+F 0 "R_C-2" H 10300 4800 50  0000 L CNN
 F 1 "150" H 10300 4600 50  0000 L CNN
 F 2 "" V 10240 4690 50  0001 C CNN
@@
 $EndComp
 $Comp
-L Device:R_US R_B-?
+L Device:R_US R_C-1
 U 1 1 61E9ABD2
 P 9600 5650
-F 0 "R_B-?" V 9805 5650 50  0000 C CNN
+F 0 "R_C-1" V 9805 5650 50  0000 C CNN
 F 1 "6.8k" V 9714 5650 50  0000 C CNN
 F 2 "" V 9640 5640 50  0001 C CNN
@@
 	10200 4400 10200 4550
 $Comp
-L Transistor_Array:ULN2803A U?
+L Transistor_Array:ULN2803A U1
 U 1 1 61C69461
 P 4800 5250
-F 0 "U?" H 4800 5817 50  0000 C CNN
+F 0 "U1" H 4800 5817 50  0000 C CNN
 F 1 "ULN2803A" H 4800 5726 50  0000 C CNN
 F 2 "" H 4850 4600 50  0001 L CNN
@@
 $EndComp
 $Comp
-L Device:Amperemeter_AC MES_B-?
+L Device:Amperemeter_AC MES_11
 U 1 1 61C983D6
 P 4800 6150
-F 0 "MES_B-?" H 5200 6200 50  0000 C CNN
+F 0 "MES_11" H 5200 6200 50  0000 C CNN
 F 1 "14.179 mA" H 5400 6050 50  0000 R CNN
 F 2 "" V 4800 6250 50  0001 C CNN
@@
 	5250 4950 5200 4950
 $Comp
-L Device:Voltmeter_DC MES?
+L Device:Voltmeter_DC MES_10
 U 1 1 61CC81A3
 P 4800 4400
-F 0 "MES?" V 5000 4650 50  0000 L CNN
+F 0 "MES_10" V 5000 4650 50  0000 L CNN
 F 1 "675.371 mV" V 5000 4000 50  0000 L CNN
 F 2 "" V 4800 4500 50  0001 C CNN
@@
 Connection ~ 5500 4400
 $Comp
-L Transistor_BJT:2N3906 Q?
+L Transistor_BJT:2N3906 Q1
 U 1 1 61D6252F
 P 5400 2300
-F 0 "Q?" H 5590 2254 50  0000 L CNN
+F 0 "Q1" H 5590 2254 50  0000 L CNN
 F 1 "2N3906" H 5590 2345 50  0000 L CNN
 F 2 "Package_TO_SOT_THT:TO-92_Inline" H 5600 2225 50  0001 L CIN
@@
 $EndComp
 $Comp
-L Device:R_US R_B-2
+L Device:R_US R4
 U 1 1 61C80CE3
 P 5500 2950
-F 0 "R_B-2" H 5600 3050 50  0000 L CNN
+F 0 "R4" H 5600 3050 50  0000 L CNN
 F 1 "150" H 5600 2850 50  0000 L CNN
 F 2 "" V 5540 2940 50  0001 C CNN
@@
 	5500 2500 5500 2600
 $Comp
-L Device:Amperemeter_AC MES_B-?
+L Device:Amperemeter_AC MES_3
 U 1 1 61D86C14
 P 4800 2300
-F 0 "MES_B-?" V 5000 2450 50  0000 C CNN
+F 0 "MES_3" V 5000 2450 50  0000 C CNN
 F 1 "139.31 uA (just saturated)" V 4600 2900 50  0000 R CNN
 F 2 "" V 4800 2400 50  0001 C CNN
@@
 	4250 2300 4250 2050
 $Comp
-L Device:R_US R_B-?
+L Device:R_US R2
 U 1 1 61DAD537
 P 4250 1400
-F 0 "R_B-?" H 4350 1500 50  0000 L CNN
+F 0 "R2" H 4350 1500 50  0000 L CNN
 F 1 "1k" H 4350 1300 50  0000 L CNN
 F 2 "" V 4290 1390 50  0001 C CNN
@@
 $EndComp
 $Comp
-L Device:R_Variable_US R?
+L Device:R_Variable_US R3
 U 1 1 61DB1117
 P 4250 1900
-F 0 "R?" H 4050 1950 50  0000 L CNN
+F 0 "R3" H 4050 1950 50  0000 L CNN
 F 1 "668/332 1k" H 4450 1950 50  0000 L CNN
 F 2 "" V 4180 1900 50  0001 C CNN
@@
 $EndComp
 $Comp
-L Device:R_US R_B-?
+L Device:R_US R1
 U 1 1 61DBDEB0
 P 3100 2300
-F 0 "R_B-?" V 3305 2300 50  0000 C CNN
+F 0 "R1" V 3305 2300 50  0000 C CNN
 F 1 "6.8k" V 3214 2300 50  0000 C CNN
 F 2 "" V 3140 2290 50  0001 C CNN
@@
 $EndComp
 $Comp
-L Device:Amperemeter_AC MES_B-?
+L Device:Amperemeter_AC MES_1
 U 1 1 61DBDEC3
 P 2000 2650
-F 0 "MES_B-?" H 1600 2500 50  0000 C CNN
+F 0 "MES_1" H 1600 2500 50  0000 C CNN
 F 1 "637.692 uA" H 1850 2750 50  0000 R CNN
 F 2 "" V 2000 2750 50  0001 C CNN
@@
 	2000 2400 2000 2450
 $Comp
-L Device:D_Schottky D?
+L Device:D_Schottky D1
 U 1 1 61DC0D35
 P 2000 2000
-F 0 "D?" V 2046 1920 50  0000 R CNN
+F 0 "D1" V 2046 1920 50  0000 R CNN
 F 1 "Schottky" V 1950 2450 50  0001 R CNN
 F 2 "" H 2000 2000 50  0001 C CNN
@@
 	2000 1750 2000 1850
 $Comp
-L Device:Amperemeter_AC MES_B-?
+L Device:Amperemeter_AC MES_2
 U 1 1 61DCD5C7
 P 3600 2300
-F 0 "MES_B-?" V 3400 2350 50  0000 C CNN
+F 0 "MES_2" V 3400 2350 50  0000 C CNN
 F 1 "637.692 uA" V 3800 2600 50  0000 R CNN
 F 2 "" V 3600 2400 50  0001 C CNN
@@
 $EndComp
 $Comp
-L Device:Voltmeter_DC MES?
+L Device:Voltmeter_DC MES_4
 U 1 1 61E5E12E
 P 6250 2300
-F 0 "MES?" H 6403 2346 50  0000 L CNN
+F 0 "MES_4" H 6403 2346 50  0000 L CNN
 F 1 "VCE 418.47 mV" H 6403 2255 50  0000 L CNN
 F 2 "" V 6250 2400 50  0001 C CNN
@@
 	5500 2600 5500 2800
 $Comp
-L Switch:SW_SPDT SW_B-?
+L Switch:SW_SPDT SW1
 U 1 1 61DBDEB6
 P 2500 2300
-F 0 "SW_B-?" H 2300 2100 50  0000 C CNN
+F 0 "SW1" H 2300 2100 50  0000 C CNN
 F 1 "SW_SPDT" H 2450 3300 50  0001 C CNN
 F 2 "" H 2500 2300 50  0001 C CNN
 F 3 "~" H 2500 2300 50  0001 C CNN
 	1    2500 2300
-	-1   0    0    -1
+	-1   0    0    1
 $EndComp
 Text Notes 3450 2050 0    50   ~ 0
